File: blinky-lights.sch (EAGLE design)
At the start: 20 parts, among them Q1 NFET, U1 555, U2 A2678EAT

Commit message: board and schematic cleanup
Parts:
- JP1: device jumper:JP1E -> blinky-lights:JP1E
- R1, R2, R3, R4, R5: device rcl:R-US_VMTB60 -> blinky-lights:RESISTOR
Connections:
- net FEEDBACK: now also R5.C; no longer R5.2
- net GND: now also R3.A; no longer R3.1
- net N$11: now also R2.A; no longer R2.1
- net N$5: now also R4.C; no longer R4.2
- net N$9: now also R1.A, R2.C; no longer R1.1, R2.2
- net REXT: now also R3.C; no longer R3.2
- net SENSE: now also R4.A; no longer R4.1
- net VCC: now also R1.C, R5.A; no longer R1.2, R5.1
Other:
- note added: "Nathan Bergey"
- note removed: "Nathan Bergey EPL"
Changed lines of the file:
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@@
 <part name="GND1" library="supply1" deviceset="GND" device=""/>
 <part name="GND3" library="supply1" deviceset="GND" device=""/>
-<part name="R3" library="rcl" deviceset="R-US_" device="VMTB60" value="500"/>
-<part name="R1" library="rcl" deviceset="R-US_" device="VMTB60" value="1k"/>
-<part name="R2" library="rcl" deviceset="R-US_" device="VMTB60" value="4k"/>
+<part name="R3" library="blinky-lights" deviceset="RESISTOR" device="" value="500"/>
+<part name="R1" library="blinky-lights" deviceset="RESISTOR" device="" value="1k"/>
+<part name="R2" library="blinky-lights" deviceset="RESISTOR" device="" value="4k"/>
 <part name="GND4" library="supply1" deviceset="GND" device=""/>
 <part name="GND5" library="supply1" deviceset="GND" device=""/>
 <part name="FRAME1" library="frames" deviceset="LETTER_L" device="" value="0.1"/>
-<part name="JP1" library="jumper" deviceset="JP1E" device="" value="5V"/>
+<part name="JP1" library="blinky-lights" deviceset="JP1E" device="" value="5V"/>
 <part name="C1" library="blinky-lights" deviceset="CAP" device="" value="0.01u"/>
 <part name="C2" library="blinky-lights" deviceset="CAP" device="" value="10u"/>
@@
 <part name="Q1" library="blinky-lights" deviceset="NFET" device=""/>
 <part name="GND8" library="supply1" deviceset="GND" device=""/>
-<part name="R4" library="rcl" deviceset="R-US_" device="VMTB60" value="10"/>
-<part name="R5" library="rcl" deviceset="R-US_" device="VMTB60" value="1k"/>
+<part name="R4" library="blinky-lights" deviceset="RESISTOR" device="" value="10"/>
+<part name="R5" library="blinky-lights" deviceset="RESISTOR" device="" value="1k"/>
 <part name="P+5" library="supply1" deviceset="VCC" device=""/>
 </parts>
@@
 <sheet>
 <plain>
-<text x="149.86" y="27.94" size="1.778" layer="97">Nathan Bergey
-EPL</text>
+<text x="149.86" y="27.94" size="2.54" layer="97">Nathan Bergey</text>
 <text x="10.16" y="154.94" size="2.54" layer="97">5V in (Hacked USB Cable)</text>
 <text x="78.74" y="152.4" size="2.54" layer="97">555 In Astable Mode
@@
 <instance part="U1" gate="G$1" x="88.9" y="93.98"/>
 <instance part="U2" gate="G$1" x="162.56" y="99.06"/>
-<instance part="LED0" gate="G$1" x="210.82" y="114.3" smashed="yes" rot="R270">
-<attribute name="NAME" x="206.248" y="110.744" size="1.778" layer="95"/>
-</instance>
-<instance part="LED2" gate="G$1" x="210.82" y="106.68" smashed="yes" rot="R270">
-<attribute name="NAME" x="206.248" y="103.124" size="1.778" layer="95"/>
-</instance>
-<instance part="LED4" gate="G$1" x="210.82" y="99.06" smashed="yes" rot="R270">
-<attribute name="NAME" x="206.248" y="95.504" size="1.778" layer="95"/>
-</instance>
-<instance part="LED7" gate="G$1" x="210.82" y="91.44" smashed="yes" rot="R270">
-<attribute name="NAME" x="206.248" y="87.884" size="1.778" layer="95"/>
-</instance>
-<instance part="LED1" gate="G$1" x="223.52" y="111.76" smashed="yes" rot="R270">
-<attribute name="NAME" x="218.948" y="108.204" size="1.778" layer="95"/>
-</instance>
-<instance part="LED3" gate="G$1" x="223.52" y="104.14" smashed="yes" rot="R270">
-<attribute name="NAME" x="218.948" y="100.584" size="1.778" layer="95"/>
-</instance>
-<instance part="LED5" gate="G$1" x="223.52" y="96.52" smashed="yes" rot="R270">
-<attribute name="NAME" x="218.948" y="92.964" size="1.778" layer="95"/>
-</instance>
-<instance part="LED6" gate="G$1" x="223.52" y="88.9" smashed="yes" rot="R270">
-<attribute name="NAME" x="218.948" y="85.344" size="1.778" layer="95"/>
-</instance>
+<instance part="LED0" gate="G$1" x="210.82" y="114.3" smashed="yes" rot="R270"/>
+<instance part="LED2" gate="G$1" x="210.82" y="106.68" smashed="yes" rot="R270"/>
+<instance part="LED4" gate="G$1" x="210.82" y="99.06" smashed="yes" rot="R270"/>
+<instance part="LED7" gate="G$1" x="210.82" y="91.44" smashed="yes" rot="R270"/>
+<instance part="LED1" gate="G$1" x="223.52" y="111.76" smashed="yes" rot="R270"/>
+<instance part="LED3" gate="G$1" x="223.52" y="104.14" smashed="yes" rot="R270"/>
+<instance part="LED5" gate="G$1" x="223.52" y="96.52" smashed="yes" rot="R270"/>
+<instance part="LED6" gate="G$1" x="223.52" y="88.9" smashed="yes" rot="R270"/>
 <instance part="P+1" gate="VCC" x="218.44" y="137.16"/>
 <instance part="P+2" gate="VCC" x="142.24" y="116.84"/>
@@
 <instance part="GND1" gate="1" x="182.88" y="71.12"/>
 <instance part="GND3" gate="1" x="22.86" y="71.12"/>
-<instance part="R3" gate="G$1" x="142.24" y="81.28" rot="R90"/>
+<instance part="R3" gate="G$1" x="142.24" y="81.28" smashed="yes" rot="R90">
+<attribute name="NAME" x="139.7" y="78.74" size="1.778" layer="95" rot="R90"/>
+<attribute name="VALUE" x="147.32" y="78.74" size="1.778" layer="96" rot="R90"/>
+</instance>
 <instance part="R1" gate="G$1" x="68.58" y="96.52" smashed="yes" rot="R90">
 <attribute name="NAME" x="67.0814" y="92.71" size="1.778" layer="95" rot="R90"/>
@@
 <attribute name="VALUE" x="193.04" y="111.252" size="1.778" layer="96" rot="R180"/>
 </instance>
-<instance part="R5" gate="G$1" x="154.94" y="129.54" rot="R270"/>
+<instance part="R5" gate="G$1" x="154.94" y="129.54" smashed="yes" rot="R270">
+<attribute name="NAME" x="157.48" y="134.62" size="1.778" layer="95" rot="R270"/>
+<attribute name="VALUE" x="157.48" y="129.54" size="1.778" layer="96" rot="R270"/>
+</instance>
 <instance part="P+5" gate="VCC" x="154.94" y="137.16"/>
 </instances>
@@
 <wire x1="144.78" y1="104.14" x2="134.62" y2="104.14" width="0.1524" layer="91"/>
 <wire x1="134.62" y1="104.14" x2="134.62" y2="124.46" width="0.1524" layer="91"/>
-<pinref part="R5" gate="G$1" pin="2"/>
+<pinref part="R5" gate="G$1" pin="C"/>
 <wire x1="134.62" y1="124.46" x2="154.94" y2="124.46" width="0.1524" layer="91"/>
 <wire x1="154.94" y1="124.46" x2="182.88" y2="124.46" width="0.1524" layer="91"/>
@@
 </segment>
 <segment>
-<pinref part="R1" gate="G$1" pin="2"/>
+<pinref part="R1" gate="G$1" pin="C"/>
 <pinref part="P+3" gate="VCC" pin="VCC"/>
 <pinref part="U1" gate="G$1" pin="RESET"/>
@@
 </segment>
 <segment>
-<pinref part="R5" gate="G$1" pin="1"/>
+<pinref part="R5" gate="G$1" pin="A"/>
 <pinref part="P+5" gate="VCC" pin="VCC"/>
 </segment>
@@
 </segment>
 <segment>
-<pinref part="R3" gate="G$1" pin="1"/>
+<pinref part="R3" gate="G$1" pin="A"/>
 <pinref part="GND4" gate="1" pin="GND"/>
 <wire x1="142.24" y1="73.66" x2="142.24" y2="76.2" width="0.1524" layer="91"/>
@@
 <net name="N$9" class="0">
 <segment>
-<pinref part="R2" gate="G$1" pin="2"/>
-<pinref part="R1" gate="G$1" pin="1"/>
+<pinref part="R2" gate="G$1" pin="C"/>
+<pinref part="R1" gate="G$1" pin="A"/>
 <pinref part="U1" gate="G$1" pin="DIS"/>
 <wire x1="68.58" y1="91.44" x2="73.66" y2="91.44" width="0.1524" layer="91"/>
@@
 <junction x="71.12" y="86.36"/>
 <pinref part="C2" gate="G$1" pin="A"/>
-<pinref part="R2" gate="G$1" pin="1"/>
+<pinref part="R2" gate="G$1" pin="A"/>
 <wire x1="71.12" y1="81.28" x2="68.58" y2="81.28" width="0.1524" layer="91"/>
 <junction x="68.58" y="81.28"/>
@@
 <segment>
 <pinref part="U2" gate="G$1" pin="REXT"/>
-<pinref part="R3" gate="G$1" pin="2"/>
+<pinref part="R3" gate="G$1" pin="C"/>
 <wire x1="144.78" y1="88.9" x2="142.24" y2="88.9" width="0.1524" layer="91"/>
 <wire x1="142.24" y1="88.9" x2="142.24" y2="86.36" width="0.1524" layer="91"/>
@@
 <segment>
 <pinref part="U2" gate="G$1" pin="OUT1"/>
-<pinref part="R4" gate="G$1" pin="2"/>
+<pinref part="R4" gate="G$1" pin="C"/>
 <wire x1="182.88" y1="109.22" x2="180.34" y2="109.22" width="0.1524" layer="91"/>
 <pinref part="Q1" gate="G$1" pin="S"/>
@@
 <wire x1="218.44" y1="111.76" x2="215.9" y2="111.76" width="0.1524" layer="91"/>
 <wire x1="215.9" y1="111.76" x2="215.9" y2="109.22" width="0.1524" layer="91"/>
-<pinref part="R4" gate="G$1" pin="1"/>
+<pinref part="R4" gate="G$1" pin="A"/>
 <wire x1="193.04" y1="109.22" x2="215.9" y2="109.22" width="0.1524" layer="91"/>
 </segment>
@@
 </sheet>
 </sheets>
-<errors>
-</errors>
 </schematic>
 </drawing>
